Commit message: wheels name changed

File: agribot_description/urdf/agribot_body.urdf.xacro (robot description, xacro)
@@ -28,5 +28,5 @@
     </link>
     <joint name="dummy_link_to_base_link" type="fixed">
-    <origin xyz="0 0 0" rpy="0 0 0" />
+    	<origin xyz="0 0 0.26" rpy="0 0 0" />
         <parent link="dummy_link"/>
         <child link="base_link"/>
@@ -67,9 +67,9 @@
 	<!--Wheels-->
     <!-- left_wheel_Back -->
-    <agribot_part parent="base_link" name="left_wheel_R"
+    <agribot_part parent="base_link" name="left_wheel_F"
           translateX="-0.2519" translateY="-0.3908" translateZ="-0.1908"
           rotateX="0.0" rotateY="0.0" rotateZ="1.57"
           color="White" />
-    <gazebo reference="left_wheel_R">
+    <gazebo reference="left_wheel_F">
         <material>Gazebo/DarkGray</material>
 	<mu1>1.0</mu1>
@@ -80,9 +80,9 @@
     </gazebo>
     <!-- left_wheel_Front -->
-    <agribot_part parent="base_link" name="left_wheel_F"
+    <agribot_part parent="base_link" name="right_wheel_F"
           translateX="-0.2519" translateY="0.3908" translateZ="-0.1908"
           rotateX="0.0" rotateY="0.0" rotateZ="1.57"
           color="White" />
-    <gazebo reference="left_wheel_F">
+    <gazebo reference="right_wheel_F">
         <material>Gazebo/DarkGray</material>
 	<mu1>1.0</mu1>
@@ -93,9 +93,9 @@
     </gazebo>
     <!-- Right_wheel_back -->
-    <agribot_part parent="base_link" name="right_wheel_R"
+    <agribot_part parent="base_link" name="left_wheel_R"
           translateX="0.2519" translateY="-0.3908" translateZ="-0.1908"
           rotateX="0.0" rotateY="0.0" rotateZ="1.57"
           color="White" />
-    <gazebo reference="right_wheel_R">
+    <gazebo reference="left_wheel_R">
         <material>Gazebo/DarkGray</material>
 	<mu1>1.0</mu1>
@@ -106,9 +106,9 @@
     </gazebo>
     <!-- Right_wheel_front -->
-    <agribot_part parent="base_link" name="right_wheel_F"
+    <agribot_part parent="base_link" name="right_wheel_R"
 	  translateX="0.2519" translateY="0.3908" translateZ="-0.1908"
           rotateX="0.0" rotateY="0.0" rotateZ="1.57"
           color="White" />
-    <gazebo reference="right_wheel_F">
+    <gazebo reference="right_wheel_R">
         <material>Gazebo/DarkGray</material>
 	<mu1>1.0</mu1>
@@ -177,5 +177,5 @@
         </inertial>
 	<collision>
-     	 <origin xyz="0 0 0" rpy="0 0 0"/>
+     	 <origin xyz="0 0 0" rpy="0 1.57 0"/>
      	 <geometry>
        		 <cylinder radius="0.03" length="0.05"/>
@@ -184,5 +184,5 @@
    	 </collision>
    	 <visual>
-    	  <origin xyz="0 0 0" rpy="0 0 0"/>
+    	  <origin xyz="0 0 0" rpy="0 1.57 0"/>
     	  <geometry>
             <cylinder radius="0.03" length="0.05"/>

Commit message: magnetometer added + bot orientation updated

File: agribot_description/urdf/agribot_body.urdf.xacro (robot description, xacro)
@@ -66,10 +66,10 @@
     </gazebo>
 	<!--Wheels-->
-    <!-- left_wheel_Back -->
-    <agribot_part parent="base_link" name="left_wheel_F"
+   <!-- left_wheel_Back -->
+    <agribot_part parent="base_link" name="left_wheel_R"
           translateX="-0.2519" translateY="-0.3908" translateZ="-0.1908"
           rotateX="0.0" rotateY="0.0" rotateZ="1.57"
           color="White" />
-    <gazebo reference="left_wheel_F">
+    <gazebo reference="left_wheel_R">
         <material>Gazebo/DarkGray</material>
 	<mu1>1.0</mu1>
@@ -79,10 +79,10 @@
   	<fdir1 value="1 0 0"/>
     </gazebo>
-    <!-- left_wheel_Front -->
-    <agribot_part parent="base_link" name="right_wheel_F"
+    <!-- right_wheel_back -->
+    <agribot_part parent="base_link" name="right_wheel_R"
           translateX="-0.2519" translateY="0.3908" translateZ="-0.1908"
           rotateX="0.0" rotateY="0.0" rotateZ="1.57"
           color="White" />
-    <gazebo reference="right_wheel_F">
+    <gazebo reference="right_wheel_R">
         <material>Gazebo/DarkGray</material>
 	<mu1>1.0</mu1>
@@ -92,10 +92,10 @@
   	<fdir1 value="1 0 0"/>
     </gazebo>
-    <!-- Right_wheel_back -->
-    <agribot_part parent="base_link" name="left_wheel_R"
+    <!-- left_wheel_front -->
+    <agribot_part parent="base_link" name="left_wheel_F"
           translateX="0.2519" translateY="-0.3908" translateZ="-0.1908"
           rotateX="0.0" rotateY="0.0" rotateZ="1.57"
           color="White" />
-    <gazebo reference="left_wheel_R">
+    <gazebo reference="left_wheel_F">
         <material>Gazebo/DarkGray</material>
 	<mu1>1.0</mu1>
@@ -106,9 +106,9 @@
     </gazebo>
     <!-- Right_wheel_front -->
-    <agribot_part parent="base_link" name="right_wheel_R"
+    <agribot_part parent="base_link" name="right_wheel_F"
 	  translateX="0.2519" translateY="0.3908" translateZ="-0.1908"
           rotateX="0.0" rotateY="0.0" rotateZ="1.57"
           color="White" />
-    <gazebo reference="right_wheel_R">
+    <gazebo reference="right_wheel_F">
         <material>Gazebo/DarkGray</material>
 	<mu1>1.0</mu1>
@@ -163,4 +163,27 @@
 <gazebo reference="gps_link">
   <material>Gazebo/Black</material>
+</gazebo>
+<link name="magnetometer_link">
+    <collision>
+      <origin xyz="0 0 0" rpy="0 0 0"/>
+      <geometry>
+        <box size="0.05 0.05 0.05"/>
+      </geometry>
+    </collision>
+    <visual>
+      <origin xyz="0 0 0" rpy="0 0 0"/>
+      <geometry>
+        <box size="0.05 0.05 0.05"/>
+      </geometry>
+      <material name="Red"/>
+    </visual>
+  </link>
+<joint name="magnetometer_to_base_link" type="fixed">
+    <origin xyz="0.3 0 0" rpy="0 0 0" />
+        <parent link="base_link"/>
+        <child link="magnetometer_link"/>
+    </joint>
+<gazebo reference="magnetometer_link">
+  <material>Gazebo/Red</material>
 </gazebo>
  <!-- Set up camera linkage and configuration -->
